Commit message: 그리퍼 TCP 오프셋을 URDF fixed joint(rg2_tcp)로 반영
두산 티칭펜던트 실측(GripperDA_v1, tool0 기준 Z 231.066mm, 회전 없음)을
onrobot_rg2_model_macro.xacro에 fixed joint/link로 추가하고, SRDF의
manipulator tip_link/end_effector를 tool0 -> rg2_tcp로 변경. MoveIt이
플랜지가 아니라 그리퍼 손끝을 직접 목표로 잡도록 해서 tool_pick_yolo_target.py의
런타임 오프셋 보정 코드를 없앴다.

File: src/cobot2_ws/m0609_rg2_bringup/urdf/onrobot_rg2_model_macro.xacro (robot description, xacro)
@@ -159,4 +159,12 @@
     <xacro:onrobot_rg2_transmission prefix="${prefix}"/>
     <xacro:onrobot_rg2_gazebo prefix="${prefix}"/>
+    <!-- 2026-07-07 두산 티칭펜던트 TCP(GripperDA_v1) 실측: effector_base 기준 회전 없이
+         Z축으로만 231.066mm. MoveIt이 그리퍼 손끝을 직접 목표로 잡도록 tip 링크로 노출. -->
+    <joint name="${prefix}tcp_joint" type="fixed">
+      <origin xyz="0 0 0.231066" rpy="0 0 0" />
+      <parent link="${effector_base}" />
+      <child link="${prefix}tcp" />
+    </joint>
+    <link name="${prefix}tcp" />
   </xacro:macro>
 </robot>

Commit message: feat: 해머 감지 시 STL 메쉬 스폰 및 파지 연동 구현, TCP/그리퍼 정렬 오류 및 충돌 회피 처리

File: src/cobot2_ws/m0609_rg2_bringup/urdf/onrobot_rg2_model_macro.xacro (robot description, xacro)
@@ -159,9 +159,9 @@
     <xacro:onrobot_rg2_transmission prefix="${prefix}"/>
     <xacro:onrobot_rg2_gazebo prefix="${prefix}"/>
-    <!-- 2026-07-07 두산 티칭펜던트 TCP(GripperDA_v1) 실측: effector_base 기준 회전 없이
+    <!-- 2026-07-07 두산 티칭펜던트 TCP(GripperDA_v1) 실측: base_link 기준 회전 없이
          Z축으로만 231.066mm. MoveIt이 그리퍼 손끝을 직접 목표로 잡도록 tip 링크로 노출. -->
     <joint name="${prefix}tcp_joint" type="fixed">
       <origin xyz="0 0 0.231066" rpy="0 0 0" />
-      <parent link="${effector_base}" />
+      <parent link="${prefix}base_link" />
       <child link="${prefix}tcp" />
     </joint>
