Commit message: feat: add physical table model to robot description and fix YAML parse exception in MoveIt launch

File: src/cobot2_ws/m0609_rg2_bringup/urdf/m0609_with_rg2.urdf.xacro (robot description, xacro)
@@ -7,3 +7,27 @@
   <!-- attaching RG2 Gripper to M0609 tool0 -->
   <xacro:onrobot_rg2 prefix="rg2_" effector_base="tool0"/>
+  <!-- 테이블 정의 (x: 1200mm, y: 650mm, z: 250mm) -->
+  <link name="table">
+    <visual>
+      <origin xyz="0 0 0" rpy="0 0 0"/>
+      <geometry>
+        <box size="1.2 0.65 0.25"/>
+      </geometry>
+      <material name="table_material">
+        <color rgba="0.6 0.6 0.6 1.0"/>
+      </material>
+    </visual>
+    <collision>
+      <origin xyz="0 0 0" rpy="0 0 0"/>
+      <geometry>
+        <box size="1.2 0.65 0.25"/>
+      </geometry>
+    </collision>
+  </link>
+  <!-- base_link에 테이블 고정 (로봇은 x=280mm에 위치, y는 중앙) -->
+  <joint name="base_to_table" type="fixed">
+    <parent link="base_link"/>
+    <child link="table"/>
+    <origin xyz="0.32 0 -0.125" rpy="0 0 0"/>
+  </joint>
 </robot>

File: src/cobot2_ws/m0609_rg2_bringup/urdf/m0609_with_rg2_camera.urdf.xacro (robot description, xacro)
@@ -9,3 +9,27 @@
   <!-- RG2 그리퍼를 tool0에 부착 -->
   <xacro:onrobot_rg2 prefix="rg2_" effector_base="tool0" has_bracket="true"/>
+  <!-- 테이블 정의 (x: 1200mm, y: 650mm, z: 250mm) -->
+  <link name="table">
+    <visual>
+      <origin xyz="0 0 0" rpy="0 0 0"/>
+      <geometry>
+        <box size="1.2 0.65 0.25"/>
+      </geometry>
+      <material name="table_material">
+        <color rgba="0.6 0.6 0.6 1.0"/>
+      </material>
+    </visual>
+    <collision>
+      <origin xyz="0 0 0" rpy="0 0 0"/>
+      <geometry>
+        <box size="1.2 0.65 0.25"/>
+      </geometry>
+    </collision>
+  </link>
+  <!-- base_link에 테이블 고정 (로봇은 x=280mm에 위치, y는 중앙) -->
+  <joint name="base_to_table" type="fixed">
+    <parent link="base_link"/>
+    <child link="table"/>
+    <origin xyz="0.32 0 -0.125" rpy="0 0 0"/>
+  </joint>
 </robot>

Commit message: Feat: 젠가 스마트 조립 및 불량 검수 시스템 성능 개선
- 첫 탐색 시작 관절 각도를 커스텀 각도 [-44.26, 18.14, 60.38, -0.02, 101.41, -36.57]로 변경
- 테이블 상면 -Y 모서리에 밀착된 1200x120x80mm 크기 컨베이어 벨트 장애물 추가
- 잘못 작성된 원판 형상의 젠가 STL을 정규 75x75x84mm 크기 직육면체 매쉬로 덮어쓰고 스폰 Z 높이를 형상 중심(Center)으로 보정
- 젠가 타워 최상면('top') 클래스 디텍션을 타겟팅하는 구면 좌표계 스캔 모션 구현
- 카메라 오프셋 역변환 및 TF 기반 gripper(tool0) 플랜지 좌표 자동 계산 헬퍼(get_tool_pose) 추가
- 로봇 한계 및 충돌 회피 실패 우회를 위해 카메라 거리(d) 및 피치(p)를 단계적으로 보정하여 IK 해를 구하는 동적 탐색 알고리즘 구현
- 스캔할 2개 촬영면 결정 시 90도 회전 관계에 있는 연속(인접) 촬영면을 우선 선택하는 알고리즘 적용
- SQLite 3 검수 결과 로깅 데이터베이스 파일 생성 및 연동 완료
- 프로젝트 규칙(AGENTS.md)에 Git 커밋 메시지 한국어 작성 조항 추가

File: src/cobot2_ws/m0609_rg2_bringup/urdf/m0609_with_rg2.urdf.xacro (robot description, xacro)
@@ -31,3 +31,27 @@
     <origin xyz="0.32 0 -0.125" rpy="0 0 0"/>
   </joint>
+  <!-- 컨베이어 벨트 정의 (X: 1200mm, Y: 120mm, Z: 80mm) -->
+  <link name="conveyor_belt">
+    <visual>
+      <origin xyz="0 0 0" rpy="0 0 0"/>
+      <geometry>
+        <mesh filename="package://m0609_rg2_bringup/meshes/conveyor_belt.stl"/>
+      </geometry>
+      <material name="conveyor_material">
+        <color rgba="0.2 0.2 0.2 1.0"/>
+      </material>
+    </visual>
+    <collision>
+      <origin xyz="0 0 0" rpy="0 0 0"/>
+      <geometry>
+        <mesh filename="package://m0609_rg2_bringup/meshes/conveyor_belt.stl"/>
+      </geometry>
+    </collision>
+  </link>
+  <!-- 테이블의 -Y 모서리 상면(+Z방향, 테이블 위)에 컨베이어 벨트 고정 -->
+  <joint name="table_to_conveyor" type="fixed">
+    <parent link="table"/>
+    <child link="conveyor_belt"/>
+    <origin xyz="0 -0.265 0.165" rpy="0 0 0"/>
+  </joint>
 </robot>

File: src/cobot2_ws/m0609_rg2_bringup/urdf/m0609_with_rg2_camera.urdf.xacro (robot description, xacro)
@@ -33,3 +33,27 @@
     <origin xyz="0.32 0 -0.125" rpy="0 0 0"/>
   </joint>
+  <!-- 컨베이어 벨트 정의 (X: 1200mm, Y: 120mm, Z: 80mm) -->
+  <link name="conveyor_belt">
+    <visual>
+      <origin xyz="0 0 0" rpy="0 0 0"/>
+      <geometry>
+        <mesh filename="package://m0609_rg2_bringup/meshes/conveyor_belt.stl"/>
+      </geometry>
+      <material name="conveyor_material">
+        <color rgba="0.2 0.2 0.2 1.0"/>
+      </material>
+    </visual>
+    <collision>
+      <origin xyz="0 0 0" rpy="0 0 0"/>
+      <geometry>
+        <mesh filename="package://m0609_rg2_bringup/meshes/conveyor_belt.stl"/>
+      </geometry>
+    </collision>
+  </link>
+  <!-- 테이블의 -Y 모서리 상면(+Z방향, 테이블 위)에 컨베이어 벨트 고정 -->
+  <joint name="table_to_conveyor" type="fixed">
+    <parent link="table"/>
+    <child link="conveyor_belt"/>
+    <origin xyz="0 -0.265 0.165" rpy="0 0 0"/>
+  </joint>
 </robot>

Commit message: Feat: 가상 천장 장애물을 URDF 및 로봇 모델에 영구 통합
- scene_builder.py의 임시 스크립트 실행 방식 대신, 테이블/컨베이어와 마찬가지로 로봇 URDF 파일(m0609_with_rg2_camera.urdf.xacro, m0609_with_rg2.urdf.xacro)에 가상 천장(ceiling) 링크 직접 추가
- robot_state_publisher 기동 시 가상 천장 장애물(2.0x2.0x0.05m)이 base_link 기준 Z=600mm 위에 항상 자동 로드되도록 설정
- scene_builder.py에서 중복 가상 천장 생성 로직 제거

File: src/cobot2_ws/m0609_rg2_bringup/urdf/m0609_with_rg2.urdf.xacro (robot description, xacro)
@@ -55,3 +55,27 @@
     <origin xyz="0 -0.265 0.165" rpy="0 0 0"/>
   </joint>
+  <!-- 가상 천장 정의 (J3 회전 범위 제한용, Z = 600mm 이상 진입 방지) -->
+  <link name="ceiling">
+    <visual>
+      <origin xyz="0 0 0" rpy="0 0 0"/>
+      <geometry>
+        <box size="2.0 2.0 0.05"/>
+      </geometry>
+      <material name="ceiling_material">
+        <color rgba="0.5 0.5 0.5 0.3"/>
+      </material>
+    </visual>
+    <collision>
+      <origin xyz="0 0 0" rpy="0 0 0"/>
+      <geometry>
+        <box size="2.0 2.0 0.05"/>
+      </geometry>
+    </collision>
+  </link>
+  <!-- 테이블 기준 Z=600mm 위에 천장 고정 (밑면이 Z=600mm에 오도록 오프셋 Z=0.75m 설정) -->
+  <joint name="table_to_ceiling" type="fixed">
+    <parent link="table"/>
+    <child link="ceiling"/>
+    <origin xyz="0 0 0.75" rpy="0 0 0"/>
+  </joint>
 </robot>

File: src/cobot2_ws/m0609_rg2_bringup/urdf/m0609_with_rg2_camera.urdf.xacro (robot description, xacro)
@@ -57,3 +57,27 @@
     <origin xyz="0 -0.265 0.165" rpy="0 0 0"/>
   </joint>
+  <!-- 가상 천장 정의 (J3 회전 범위 제한용, Z = 600mm 이상 진입 방지) -->
+  <link name="ceiling">
+    <visual>
+      <origin xyz="0 0 0" rpy="0 0 0"/>
+      <geometry>
+        <box size="2.0 2.0 0.05"/>
+      </geometry>
+      <material name="ceiling_material">
+        <color rgba="0.5 0.5 0.5 0.3"/>
+      </material>
+    </visual>
+    <collision>
+      <origin xyz="0 0 0" rpy="0 0 0"/>
+      <geometry>
+        <box size="2.0 2.0 0.05"/>
+      </geometry>
+    </collision>
+  </link>
+  <!-- 테이블 기준 Z=600mm 위에 천장 고정 (밑면이 Z=600mm에 오도록 오프셋 Z=0.75m 설정) -->
+  <joint name="table_to_ceiling" type="fixed">
+    <parent link="table"/>
+    <child link="ceiling"/>
+    <origin xyz="0 0 0.75" rpy="0 0 0"/>
+  </joint>
 </robot>

Commit message: Feat: 가상 천장 높이를 Z=1000mm로 수정
- 기존 Z=600mm 가상 천장이 너무 낮아 작업 영역을 제한할 우려가 있어 Z=1000mm로 높이 조정
- table_to_ceiling 고정 조인트의 Z축 오프셋을 0.75m에서 1.15m로 수정

File: src/cobot2_ws/m0609_rg2_bringup/urdf/m0609_with_rg2.urdf.xacro (robot description, xacro)
@@ -55,5 +55,5 @@
     <origin xyz="0 -0.265 0.165" rpy="0 0 0"/>
   </joint>
-  <!-- 가상 천장 정의 (J3 회전 범위 제한용, Z = 600mm 이상 진입 방지) -->
+  <!-- 가상 천장 정의 (J3 회전 범위 제한용, Z = 1000mm 이상 진입 방지) -->
   <link name="ceiling">
     <visual>
@@ -73,9 +73,9 @@
     </collision>
   </link>
-  <!-- 테이블 기준 Z=600mm 위에 천장 고정 (밑면이 Z=600mm에 오도록 오프셋 Z=0.75m 설정) -->
+  <!-- 테이블 기준 Z=1000mm 위에 천장 고정 (밑면이 Z=1000mm에 오도록 오프셋 Z=1.15m 설정) -->
   <joint name="table_to_ceiling" type="fixed">
     <parent link="table"/>
     <child link="ceiling"/>
-    <origin xyz="0 0 0.75" rpy="0 0 0"/>
+    <origin xyz="0 0 1.15" rpy="0 0 0"/>
   </joint>
 </robot>

File: src/cobot2_ws/m0609_rg2_bringup/urdf/m0609_with_rg2_camera.urdf.xacro (robot description, xacro)
@@ -57,5 +57,5 @@
     <origin xyz="0 -0.265 0.165" rpy="0 0 0"/>
   </joint>
-  <!-- 가상 천장 정의 (J3 회전 범위 제한용, Z = 600mm 이상 진입 방지) -->
+  <!-- 가상 천장 정의 (J3 회전 범위 제한용, Z = 1000mm 이상 진입 방지) -->
   <link name="ceiling">
     <visual>
@@ -75,9 +75,9 @@
     </collision>
   </link>
-  <!-- 테이블 기준 Z=600mm 위에 천장 고정 (밑면이 Z=600mm에 오도록 오프셋 Z=0.75m 설정) -->
+  <!-- 테이블 기준 Z=1000mm 위에 천장 고정 (밑면이 Z=1000mm에 오도록 오프셋 Z=1.15m 설정) -->
   <joint name="table_to_ceiling" type="fixed">
     <parent link="table"/>
     <child link="ceiling"/>
-    <origin xyz="0 0 0.75" rpy="0 0 0"/>
+    <origin xyz="0 0 1.15" rpy="0 0 0"/>
   </joint>
 </robot>

Commit message: Feat: 가상 천장 높이를 Z=800mm로 재보정
- Z=1000mm 높이가 실 하드웨어 세이프 영역 대비 높아, 보다 정밀한 천장 간섭 회피를 위해 Z=800mm로 조정
- table_to_ceiling 고정 조인트 Z축 오프셋을 1.15m에서 0.95m로 수정

File: src/cobot2_ws/m0609_rg2_bringup/urdf/m0609_with_rg2.urdf.xacro (robot description, xacro)
@@ -55,5 +55,5 @@
     <origin xyz="0 -0.265 0.165" rpy="0 0 0"/>
   </joint>
-  <!-- 가상 천장 정의 (J3 회전 범위 제한용, Z = 1000mm 이상 진입 방지) -->
+  <!-- 가상 천장 정의 (J3 회전 범위 제한용, Z = 800mm 이상 진입 방지) -->
   <link name="ceiling">
     <visual>
@@ -73,9 +73,9 @@
     </collision>
   </link>
-  <!-- 테이블 기준 Z=1000mm 위에 천장 고정 (밑면이 Z=1000mm에 오도록 오프셋 Z=1.15m 설정) -->
+  <!-- 테이블 기준 Z=800mm 위에 천장 고정 (밑면이 Z=800mm에 오도록 오프셋 Z=0.95m 설정) -->
   <joint name="table_to_ceiling" type="fixed">
     <parent link="table"/>
     <child link="ceiling"/>
-    <origin xyz="0 0 1.15" rpy="0 0 0"/>
+    <origin xyz="0 0 0.95" rpy="0 0 0"/>
   </joint>
 </robot>

File: src/cobot2_ws/m0609_rg2_bringup/urdf/m0609_with_rg2_camera.urdf.xacro (robot description, xacro)
@@ -57,5 +57,5 @@
     <origin xyz="0 -0.265 0.165" rpy="0 0 0"/>
   </joint>
-  <!-- 가상 천장 정의 (J3 회전 범위 제한용, Z = 1000mm 이상 진입 방지) -->
+  <!-- 가상 천장 정의 (J3 회전 범위 제한용, Z = 800mm 이상 진입 방지) -->
   <link name="ceiling">
     <visual>
@@ -75,9 +75,9 @@
     </collision>
   </link>
-  <!-- 테이블 기준 Z=1000mm 위에 천장 고정 (밑면이 Z=1000mm에 오도록 오프셋 Z=1.15m 설정) -->
+  <!-- 테이블 기준 Z=800mm 위에 천장 고정 (밑면이 Z=800mm에 오도록 오프셋 Z=0.95m 설정) -->
   <joint name="table_to_ceiling" type="fixed">
     <parent link="table"/>
     <child link="ceiling"/>
-    <origin xyz="0 0 1.15" rpy="0 0 0"/>
+    <origin xyz="0 0 0.95" rpy="0 0 0"/>
   </joint>
 </robot>

Commit message: 로봇 후방 가상 안전 충돌 벽(safety_wall) 정의 추가

File: src/cobot2_ws/m0609_rg2_bringup/urdf/m0609_with_rg2.urdf.xacro (robot description, xacro)
@@ -79,3 +79,28 @@
     <origin xyz="0 0 0.95" rpy="0 0 0"/>
   </joint>
+  <!-- 로봇 뒤편 안전 가상 벽 정의 (배선 걸림 및 J3, J4 후방 회전 방지용) -->
+  <link name="safety_wall">
+    <visual>
+      <origin xyz="0 0 0" rpy="0 0 0"/>
+      <geometry>
+        <!-- 두께 2cm, 가로 100cm, 높이 120cm 박스 -->
+        <box size="0.02 1.0 1.2"/>
+      </geometry>
+      <material name="wall_material">
+        <color rgba="0.8 0.1 0.1 0.3"/> <!-- 반투명 빨간색으로 시각화 -->
+      </material>
+    </visual>
+    <collision>
+      <origin xyz="0 0 0" rpy="0 0 0"/>
+      <geometry>
+        <box size="0.02 1.0 1.2"/>
+      </geometry>
+    </collision>
+  </link>
+  <!-- base_link 기준 X = -35cm 뒤쪽, Z = 50cm 높이에 벽의 중심이 오도록 고정 -->
+  <joint name="base_to_safety_wall" type="fixed">
+    <parent link="base_link"/>
+    <child link="safety_wall"/>
+    <origin xyz="-0.35 0 0.5" rpy="0 0 0"/>
+  </joint>
 </robot>

File: src/cobot2_ws/m0609_rg2_bringup/urdf/m0609_with_rg2_camera.urdf.xacro (robot description, xacro)
@@ -81,3 +81,28 @@
     <origin xyz="0 0 0.95" rpy="0 0 0"/>
   </joint>
+  <!-- 로봇 뒤편 안전 가상 벽 정의 (배선 걸림 및 J3, J4 후방 회전 방지용) -->
+  <link name="safety_wall">
+    <visual>
+      <origin xyz="0 0 0" rpy="0 0 0"/>
+      <geometry>
+        <!-- 두께 2cm, 가로 100cm, 높이 120cm 박스 -->
+        <box size="0.02 1.0 1.2"/>
+      </geometry>
+      <material name="wall_material">
+        <color rgba="0.8 0.1 0.1 0.3"/> <!-- 반투명 빨간색으로 시각화 -->
+      </material>
+    </visual>
+    <collision>
+      <origin xyz="0 0 0" rpy="0 0 0"/>
+      <geometry>
+        <box size="0.02 1.0 1.2"/>
+      </geometry>
+    </collision>
+  </link>
+  <!-- base_link 기준 X = -35cm 뒤쪽, Z = 50cm 높이에 벽의 중심이 오도록 고정 -->
+  <joint name="base_to_safety_wall" type="fixed">
+    <parent link="base_link"/>
+    <child link="safety_wall"/>
+    <origin xyz="-0.35 0 0.5" rpy="0 0 0"/>
+  </joint>
 </robot>

Commit message: 안전성 최적화: JReady 시작위치 변경, J3 각제한 완화(±100도) 및 천장높이 재조정(900mm)

File: src/cobot2_ws/m0609_rg2_bringup/urdf/m0609_with_rg2.urdf.xacro (robot description, xacro)
@@ -73,9 +73,9 @@
     </collision>
   </link>
-  <!-- 테이블 기준 Z=800mm 위에 천장 고정 (밑면이 Z=800mm에 오도록 오프셋 Z=0.95m 설정) -->
+  <!-- 테이블 기준 Z=900mm 위에 천장 고정 (밑면이 Z=900mm에 오도록 오프셋 Z=1.05m 설정) -->
   <joint name="table_to_ceiling" type="fixed">
     <parent link="table"/>
     <child link="ceiling"/>
-    <origin xyz="0 0 0.95" rpy="0 0 0"/>
+    <origin xyz="0 0 1.05" rpy="0 0 0"/>
   </joint>
   <!-- 로봇 뒤편 안전 가상 벽 정의 (배선 걸림 및 J3, J4 후방 회전 방지용) -->

File: src/cobot2_ws/m0609_rg2_bringup/urdf/m0609_with_rg2_camera.urdf.xacro (robot description, xacro)
@@ -75,9 +75,9 @@
     </collision>
   </link>
-  <!-- 테이블 기준 Z=800mm 위에 천장 고정 (밑면이 Z=800mm에 오도록 오프셋 Z=0.95m 설정) -->
+  <!-- 테이블 기준 Z=900mm 위에 천장 고정 (밑면이 Z=900mm에 오도록 오프셋 Z=1.05m 설정) -->
   <joint name="table_to_ceiling" type="fixed">
     <parent link="table"/>
     <child link="ceiling"/>
-    <origin xyz="0 0 0.95" rpy="0 0 0"/>
+    <origin xyz="0 0 1.05" rpy="0 0 0"/>
   </joint>
   <!-- 로봇 뒤편 안전 가상 벽 정의 (배선 걸림 및 J3, J4 후방 회전 방지용) -->
